Commit message: Comprehensive update to EZGripper ROS2 package
This commit includes multiple improvements to the EZGripper ROS2 package:

1. Fixed joint state publishing for triple gripper configuration:
   - Ensured all knuckle joints are properly published for all grippers
   - Used URDF naming conventions as the source of truth instead of TF tree detection
   - Created appropriate subscribers for each gripper's command topics

2. Improved launch files:
   - Updated triple gripper launch files for better configuration and testing
   - Added debug launch files for troubleshooting
   - Removed obsolete display launch files
   - Ensured consistent parameter passing across all launch files

3. Enhanced URDF files:
   - Improved triple gripper configuration with proper instantiation of single grippers
   - Fixed orientation and positioning issues
   - Ensured consistent naming conventions

4. Added process management:
   - Added cleanup scripts to handle lingering processes
   - Integrated cleanup into launch files for better robustness

5. Added documentation:
   - Created PARAMETERS_AND_NAMING.md for parameter documentation
   - Added testing and orientation guides for triple gripper

These changes ensure that the EZGripper package works correctly with all gripper configurations, especially the triple gripper setup, and provides better documentation and tools for debugging and testing.

File: ezgripper_description/urdf/SAKE_double_mount.urdf.xacro (robot description, xacro)
@@ -17,4 +17,5 @@
 				</geometry>
 				<material name="blue"/>
+				<!-- Using material defined in materials.urdf.xacro -->
 			</visual>
 			<collision>

File: ezgripper_description/urdf/SAKE_single_mount.urdf.xacro (robot description, xacro)
@@ -1,6 +1,5 @@
 <?xml version="1.0" encoding="UTF-8"?>
 <robot name="SAKE_single_mount" xmlns:xacro="http://ros.org/wiki/xacro">
-    <!-- Include centralized material definitions (properties only) -->
-    <xacro:include filename="$(find ezgripper_description)/urdf/materials.xacro" />
+    <!-- Material definitions are included in the parent file -->
 	<xacro:macro name="SAKE_single_mount" params="prefix parent_link *origin">
 		<!-- links -->

File: ezgripper_description/urdf/SAKE_triple_mount.urdf.xacro (robot description, xacro)
@@ -16,5 +16,6 @@
 					<mesh filename="package://ezgripper_description/meshes/visual/SAKE_Triple_Mount.stl"/>
 				</geometry>
-				<material name="ezgripper_blue"/>
+				<material name="blue"/>
+				<!-- Using material defined in materials.urdf.xacro -->
 			</visual>
 			<collision>

File: ezgripper_description/urdf/ezgripper_double_with_mount_standalone.urdf.xacro (robot description, xacro)
@@ -1,8 +1,14 @@
 <?xml version="1.0" encoding="UTF-8"?>
 <robot name="ezgripper_single_mount_instantiation" xmlns:xacro="http://ros.org/wiki/xacro">
-    <xacro:property name="prefix" value="left" />
+    <!-- Robot prefix parameter for consistent naming across all components -->
+    <xacro:arg name="prefix" default="PrefixDefault"/>
+    <!-- Double gripper uses fixed unit numbers: 1 for gripper1, 2 for gripper2 -->
+    <xacro:property name="prefix" value="$(arg prefix)" />
     <xacro:property name="ezgripper_offset_x" value="0.00"/>
     <xacro:property name="ezgripper_offset_y" value="0.0"/>
     <xacro:property name="ezgripper_offset_z" value="0.0"/>
+    <xacro:include filename="$(find ezgripper_description)/urdf/materials.urdf.xacro" />
+    <!-- Define materials -->
+    <xacro:define_ezgripper_materials />
     <xacro:include filename="ezgripper_double_with_mount.urdf.xacro" />
     <!-- Instantiate the gripper and mount assembly with specified parameters -->
@@ -21,5 +27,5 @@
             </geometry>
             <origin rpy="0 0 0" xyz="0 0 0.21"/>
-            <material name="black"/>
+            <material name="ezgripper_black"/>
         </visual>
         <collision>

File: ezgripper_description/urdf/ezgripper_single.urdf.xacro (robot description, xacro)
@@ -1,6 +1,5 @@
 <?xml version="1.0" encoding="UTF-8"?>
 <robot name="ezgripper_single" xmlns:xacro="http://ros.org/wiki/xacro">
-    <!-- Include centralized material definitions (properties only) -->
-    <xacro:include filename="$(find ezgripper_description)/urdf/materials.xacro" />
+    <!-- Material definitions are included in the parent file -->
 	<xacro:macro name="ezgripper_single" params="prefix parent_link *origin">
 		<!-- links -->

File: ezgripper_description/urdf/ezgripper_single_mount.urdf.xacro (robot description, xacro)
@@ -9,5 +9,5 @@
 					<mesh filename="file://$(find ezgripper_description)/meshes/visual/SAKE_Single_Mount.stl"/>
 				</geometry>
-				<material name="blue"/>
+				<material name="ezgripper_blue"/>
 			</visual>
 			<collision>
@@ -43,5 +43,5 @@
 					<mesh filename="file://$(find ezgripper_description)/meshes/visual/SAKE_Palm_IM.stl"/>
 				</geometry>
-				<material name="blue"/>
+				<material name="ezgripper_blue"/>
 			</visual>
 			<collision>
@@ -90,5 +90,5 @@
 					<mesh filename="file://$(find ezgripper_description)/meshes/visual/SAKE_Finger_L1_IM.stl"/>
 				</geometry>
-				<material name="grey"/>
+				<material name="ezgripper_grey"/>
 			</visual>
 			<collision>
@@ -114,5 +114,5 @@
 					<mesh filename="file://$(find ezgripper_description)/meshes/visual/SAKE_Finger_L2_IM.stl"/>
 				</geometry>
-				<material name="grey"/>
+				<material name="ezgripper_grey"/>
 			</visual>
 			<collision>
@@ -138,5 +138,5 @@
 					<mesh filename="file://$(find ezgripper_description)/meshes/visual/SAKE_Finger_Pad_IM.stl"/>
 				</geometry>
-				<material name="grey"/>
+				<material name="ezgripper_grey"/>
 			</visual>
 			<collision>
@@ -209,5 +209,5 @@
       <plugin>gazebo_ros2_control/GazeboSystem</plugin>
     </hardware>
-		<joint name="left_ezgripper_knuckle_palm_L1_1">
+		<joint name="${prefix}_ezgripper_knuckle_palm_L1_1">
       <command_interface name="position"/>
       <state_interface name="position"/>
@@ -215,6 +215,6 @@
       <state_interface name="effort"/>
     </joint>
-    <joint name="left_ezgripper_knuckle_palm_L1_2">
-			<param name="mimic">left_ezgripper_knuckle_palm_L1_1</param>
+    <joint name="${prefix}_ezgripper_knuckle_palm_L1_2">
+			<param name="mimic">${prefix}_ezgripper_knuckle_palm_L1_1</param>
 			<param name="multiplier">1</param>
 			<command_interface name="position"/>

File: ezgripper_description/urdf/ezgripper_single_mount_standalone.urdf.xacro (robot description, xacro)
@@ -5,7 +5,14 @@
 	<xacro:property name="ezgripper_offset_z" value="0.3"/>
 	<xacro:include filename="$(find ezgripper_description)/urdf/materials.urdf.xacro"/>
+	<!-- Define materials -->
+	<xacro:define_ezgripper_materials />
+	<xacro:include filename="$(find ezgripper_description)/urdf/ezgripper_single.urdf.xacro"/>
 	<xacro:include filename="$(find ezgripper_description)/urdf/ezgripper_single_mount.urdf.xacro"/>
+	<!-- Robot prefix parameter for consistent naming across all components -->
+	<xacro:arg name="prefix" default="ezgripper_1"/>
+	<!-- Define the prefix property to ensure it's accessible in all included files -->
+	<xacro:property name="prefix" value="$(arg prefix)"/>
 	<!-- Add the gripper -->
-	<xacro:ezgripper_single_mount prefix="left" parent_link="base_link">
+	<xacro:ezgripper_single_mount prefix="$(arg prefix)" parent_link="base_link">
 		<origin xyz="${ezgripper_offset_x} ${ezgripper_offset_y} ${ezgripper_offset_z}" rpy="0 0 0"/>
 	</xacro:ezgripper_single_mount>
@@ -21,5 +28,5 @@
 			</geometry>
 			<origin rpy="0 0 0" xyz="0 0 0.21"/>
-			<material name="black"/>
+			<material name="ezgripper_black"/>
 		</visual>
 		<collision>

File: ezgripper_description/urdf/ezgripper_single_with_mount.urdf.xacro (robot description, xacro)
@@ -1,6 +1,5 @@
 <?xml version="1.0" encoding="UTF-8"?>
 <robot name="ezgripper_single_with_mount" xmlns:xacro="http://ros.org/wiki/xacro">
-    <!-- Include centralized material definitions (properties only) -->
-    <xacro:include filename="$(find ezgripper_description)/urdf/materials.xacro" />
+    <!-- Material definitions are included in the parent file -->
     <xacro:macro name="ezgripper_single_with_mount" params="prefix parent_link *origin">
 	<!-- Include the gripper and mount files -->

File: ezgripper_description/urdf/ezgripper_single_with_mount_standalone.urdf.xacro (robot description, xacro)
@@ -2,7 +2,10 @@
 <robot name="ezgripper_single_mount_instantiation" xmlns:xacro="http://ros.org/wiki/xacro">
     <!-- Include centralized material definitions -->
-    <xacro:include filename="$(find ezgripper_description)/urdf/materials.xacro" />
+    <xacro:include filename="$(find ezgripper_description)/urdf/materials.urdf.xacro" />
+    <!-- Define materials -->
     <xacro:define_ezgripper_materials />
-    <xacro:property name="prefix" value="left" />
+    <!-- Robot prefix parameter for consistent naming across all components -->
+    <xacro:arg name="prefix" default="PrefixDefault"/>
+    <xacro:property name="prefix" value="$(arg prefix)" />
     <xacro:property name="ezgripper_offset_x" value="0.00"/>
     <xacro:property name="ezgripper_offset_y" value="0.0"/>

File: ezgripper_description/urdf/ezgripper_triple_with_mount.urdf.xacro (robot description, xacro)
@@ -2,4 +2,6 @@
 <robot name="ezgripper_triple_with_mount" xmlns:xacro="http://ros.org/wiki/xacro">
   <xacro:macro name="ezgripper_triple_with_mount" params="prefix parent_link *origin">
+    <!-- Use the robot prefix for consistent naming across all components -->
+    <!-- Define gripper spacing properties -->
     <xacro:property name="gripper_spacing" value="0.068"/>  <!-- Gripper separation in m (6.8cm) -->
     <xacro:property name="gripper_offset" value="0.01254"/>   <!-- Gripper offset in the positive X direction from the mount in m (1.254cm) -->
@@ -7,18 +9,19 @@
     <xacro:include filename="$(find ezgripper_description)/urdf/SAKE_triple_mount.urdf.xacro" />
     <xacro:include filename="$(find ezgripper_description)/urdf/ezgripper_single.urdf.xacro" />
-    <!-- Instantiate the triple mount -->
+    <!-- Instantiate the triple mount as a common component for all grippers -->
     <xacro:SAKE_triple_mount prefix="${prefix}" parent_link="${parent_link}">
       <xacro:insert_block name="origin"/>
     </xacro:SAKE_triple_mount>
-    <!-- Instantiate the first ezgripper_single -->
-    <xacro:ezgripper_single prefix="${prefix}_gripper1" parent_link="${prefix}_ezgripper_to_mount">
+    <!-- Instantiate the first ezgripper (left position) with unique prefix -->
+    <!-- Each gripper in the triple assembly has a unique prefix to ensure proper naming -->
+    <xacro:ezgripper_single prefix="${prefix}_1" parent_link="${prefix}_ezgripper_to_mount">
       <origin xyz="${gripper_offset} 0 ${gripper_spacing}" rpy="0 0 0"/>
     </xacro:ezgripper_single>
-    <!-- Instantiate the second ezgripper_single -->
-    <xacro:ezgripper_single prefix="${prefix}_gripper2" parent_link="${prefix}_ezgripper_to_mount">
+    <!-- Instantiate the second ezgripper (center position) with unique prefix -->
+    <xacro:ezgripper_single prefix="${prefix}_2" parent_link="${prefix}_ezgripper_to_mount">
       <origin xyz="${gripper_offset} 0 0" rpy="0 0 0"/>
     </xacro:ezgripper_single>
-    <!-- Instantiate the third ezgripper_single -->
-    <xacro:ezgripper_single prefix="${prefix}_gripper3" parent_link="${prefix}_ezgripper_to_mount">
+    <!-- Instantiate the third ezgripper (right position) with unique prefix -->
+    <xacro:ezgripper_single prefix="${prefix}_3" parent_link="${prefix}_ezgripper_to_mount">
       <origin xyz="${gripper_offset} 0 -${gripper_spacing}" rpy="0 0 0"/>
     </xacro:ezgripper_single>

File: ezgripper_description/urdf/ezgripper_triple_with_mount_standalone.urdf.xacro (robot description, xacro)
@@ -1,14 +1,24 @@
 <?xml version="1.0" encoding="UTF-8"?>
 <robot name="ezgripper_triple_mount_instantiation" xmlns:xacro="http://ros.org/wiki/xacro">
+    <!-- Arm name parameter for consistent naming across all components -->
+    <xacro:arg name="prefix" default="left_arm"/>
+    <!-- Define the prefix property to ensure it's accessible in all included files -->
+    <xacro:property name="prefix" value="$(arg prefix)"/>
+    <!-- Triple gripper uses fixed unit numbers: 1 for left, 2 for center, 3 for right -->
+    <!-- Triple gripper uses fixed unit numbers: 1 for left, 2 for center, 3 for right -->
     <!-- Include centralized material definitions -->
-    <xacro:include filename="$(find ezgripper_description)/urdf/materials.xacro" />
+    <xacro:include filename="$(find ezgripper_description)/urdf/materials.urdf.xacro" />
+    <!-- Define materials -->
     <xacro:define_ezgripper_materials />
-    <xacro:property name="prefix" value="left" />
     <xacro:property name="ezgripper_offset_x" value="0.00"/>
     <xacro:property name="ezgripper_offset_y" value="0.0"/>
     <xacro:property name="ezgripper_offset_z" value="0.21"/>
+    <!-- Include the triple gripper with mount XACRO file -->
     <xacro:include filename="ezgripper_triple_with_mount.urdf.xacro" />
     <!-- Instantiate the gripper and mount assembly with specified parameters -->
-    <xacro:ezgripper_triple_with_mount prefix="${prefix}" parent_link="base_link">
+    <!-- The triple gripper uses the arm name as prefix and fixed unit numbers (1,2,3) for each gripper position -->
+    <xacro:ezgripper_triple_with_mount
+        prefix="$(arg prefix)"
+        parent_link="base_link">
         <origin xyz="${ezgripper_offset_x} ${ezgripper_offset_y} ${ezgripper_offset_z}" rpy="0 0 0"/>
     </xacro:ezgripper_triple_with_mount>

File: ezgripper_description/urdf/materials.urdf.xacro (robot description, xacro)
@@ -1,15 +1,23 @@
 <?xml version="1.0"?>
 <robot xmlns:xacro="http://ros.org/wiki/xacro">
-  <material name="black">
-    <color rgba="0.0 0.0 0.0 1.0"/>
-  </material>
-  <material name="blue">
-    <color rgba="0.0 0.0 0.8 1.0"/>
-  </material>
-  <material name="grey">
-    <color rgba="0.5 0.5 0.5 1"/>
-  </material>
-  <material name="white">
-    <color rgba="1.0 1.0 1.0 1.0"/> <!-- RGBA: Red, Green, Blue, Alpha (transparency) -->
-  </material>
+  <!-- EZGripper material color properties -->
+  <xacro:property name="ezgripper_black_rgba" value="0.0 0.0 0.0 1.0" />
+  <xacro:property name="ezgripper_blue_rgba" value="0.0 0.0 0.8 1.0" />
+  <xacro:property name="ezgripper_grey_rgba" value="0.5 0.5 0.5 1.0" />
+  <xacro:property name="ezgripper_white_rgba" value="1.0 1.0 1.0 1.0" />
+  <!-- EZGripper material definitions macro -->
+  <xacro:macro name="define_ezgripper_materials">
+    <material name="ezgripper_black">
+      <color rgba="${ezgripper_black_rgba}"/>
+    </material>
+    <material name="ezgripper_blue">
+      <color rgba="${ezgripper_blue_rgba}"/>
+    </material>
+    <material name="ezgripper_grey">
+      <color rgba="${ezgripper_grey_rgba}"/>
+    </material>
+    <material name="ezgripper_white">
+      <color rgba="${ezgripper_white_rgba}"/>
+    </material>
+  </xacro:macro>
 </robot>
